File: kicad/main/kicad.kicad_sch (KiCad schematic)
At the start: 30 parts, among them J1 5V, J2 Cal Z, J3 Cal Y, J4 CAL X, J6 Conn_01x05_Female, J7 Conn_01x01_Male, J9 C1, Q1 SI2302, Q2 SI2302, Q3 SI2302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

Commit message: Updates
Parts:
- J1: symbol Connector:Conn_01x02_Female -> Connector:Conn_01x02_Socket
- J2, J3, J4: symbol Connector:Conn_01x04_Female -> Connector:Conn_01x04_Socket
- J6: symbol Connector:Conn_01x05_Female -> Connector:Conn_01x05_Socket
- J7: symbol Connector:Conn_01x01_Male -> Connector:Conn_01x01_Pin
- J9: symbol Connector:Conn_01x04_Male -> Connector:Conn_01x04_Pin
Connections:
- net +3V3 renamed +3.3V
Other:
- moved on the sheet: C1, C2, J1, J6, J7, J9, Q1, Q2, R1, R5, R6, R9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
